File: QMK 100 FRL/untitled.kicad_sch (KiCad schematic)
At the start: 203 parts

Commit message: Changed MCU
Changed MCU from ATMEL AT90USB1286-AUR to ATMEGA128A-AU which is the newest version.
Parts:
- gave numbers to parts that had none: 203
Other:
- moved on the sheet: D1, D10, D11, D12, D13, D14, D15, D16, D17, D18, D19, D2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
