File: QMK 100 FRL/matrix.kicad_sch (KiCad schematic)
At the start: 299 parts

Commit message: Finished from the first schema and pcb
Finished the schematics and foot prints links and updated the pcb foot prints to the pcb.
Parts:
- removed R?: 1K, Resistor_SMD:R_0603_1608Metric, symbol Device:R_Small
- added R16, R18, R43: 1K, Resistor_SMD:R_0603_1608Metric, symbol Device:R_Small
- MX_LALT1: renamed from MX_LALT?; footprint MX_Alps_Hybrid:MX-1.5U -> MX_Alps_Hybrid:MX-1.25U
- MX_LCTRL1: renamed from MX_LCTRL?; footprint MX_Alps_Hybrid:MX-1.5U -> MX_Alps_Hybrid:MX-1.25U
- MX_LWIN1: renamed from MX_LWIN?; footprint MX_Alps_Hybrid:MX-1.5U -> MX_Alps_Hybrid:MX-1U
- MX_Num_+_2U1: renamed from MX_Num_+_2U; footprint MX_Alps_Hybrid:MX-1U -> MX_Alps_Hybrid:MX-2U
- MX_Num_0_2U1: renamed from MX_Num_0_2U; footprint MX_Alps_Hybrid:MX-1U -> MX_Alps_Hybrid:MX-2U
- MX_Num_Enter_2U1: renamed from MX_Num_Enter_2U; footprint MX_Alps_Hybrid:MX-1U -> MX_Alps_Hybrid:MX-2U
- MX_RALT1: renamed from MX_RALT?; footprint MX_Alps_Hybrid:MX-1.5U -> MX_Alps_Hybrid:MX-1.25U
- MX_RCTRL1: renamed from MX_RCTRL?; footprint MX_Alps_Hybrid:MX-1.5U -> MX_Alps_Hybrid:MX-1.25U
- MX_RFn1: renamed from MX_RFn?; footprint MX_Alps_Hybrid:MX-1.5U -> MX_Alps_Hybrid:MX-1.25U
- MX_RWIN1: renamed from MX_RWIN?; footprint MX_Alps_Hybrid:MX-1.5U -> MX_Alps_Hybrid:MX-1.25U
- MX_SP6.25U1: renamed from MX_SP6.25U?; footprint MX_Alps_Hybrid:MX-10U -> MX_Alps_Hybrid:MX-6.25U
- gave numbers to parts that had none: 260
- renumbered MX_LALT7U to MX_LALT7U1, MX_LCTRL7U to MX_LCTRL7U1, MX_LWIN7U to MX_LWIN7U1, MX_Num_* to MX_Num_*1, MX_Num_+ to MX_Num_+1, MX_Num_- to MX_Num_-1, MX_Num_. to MX_Num_.1, MX_Num_/ to MX_Num_/1, MX_Num_7 to MX_Num_1, MX_Num_00 to MX_Num_10, MX_Num_0 to MX_Num_11, MX_Num_8 to MX_Num_2, MX_Num_9 to MX_Num_3, MX_Num_1 to MX_Num_7, MX_Num_2 to MX_Num_8, MX_Num_3 to MX_Num_9, MX_Num_L to MX_Num_L1, MX_RALT7U to MX_RALT7U1, MX_RCTRL7U to MX_RCTRL7U1, MX_RWIN7U to MX_RWIN7U1, MX_SP7U to MX_SP7U1
Connections:
- net +5V: now also MX_LALT7U1.3 (LED), MX_LCTRL7U1.3 (LED), MX_Num_*1.3 (LED), MX_Num_+1.3 (LED), MX_Num_+_2U1.3 (LED), MX_Num_-1.3 (LED), MX_Num_-2.3 (LED), MX_Num_.1.3 (LED), MX_Num_/1.3 (LED), MX_Num_0_2U1.3 (LED), MX_Num_1.3 (LED), MX_Num_10.3 (LED), MX_Num_11.1 (COL), MX_Num_11.3 (LED), MX_Num_2.3 (LED), MX_Num_3.3 (LED), MX_Num_4.3 (LED), MX_Num_5.3 (LED), MX_Num_6.3 (LED), MX_Num_7.3 (LED), MX_Num_8.3 (LED), MX_Num_9.3 (LED), MX_Num_Enter_2U1.3 (LED), MX_Num_L1.3 (LED), MX_Num_Macro1.3 (LED), MX_Num_Macro2.3 (LED), MX_RALT1.3 (LED), MX_RALT7U1.3 (LED), MX_RCTRL7U1.3 (LED), MX_RFn1.3 (LED), MX_RWIN1.3 (LED), MX_RWIN7U1.3 (LED)
- net COL0: now also MX_LCTRL7U1.1 (COL), MX_LWIN1.1 (COL), MX_LWIN7U1.1 (COL)
- net COL1: now also MX_LALT7U1.1 (COL)
- net COL10: now also MX_Num_+1.1 (COL), MX_Num_+_2U1.1 (COL), MX_Num_-1.1 (COL), MX_Num_-2.1 (COL), MX_Num_Enter_2U1.1 (COL), MX_Num_Macro1.1 (COL), MX_Num_Macro2.1 (COL)
- net COL5: now also MX_RALT1.1 (COL), MX_RALT7U1.1 (COL), MX_RFn1.1 (COL)
- net COL6: now also MX_RCTRL7U1.1 (COL), MX_RWIN1.1 (COL), MX_RWIN7U1.1 (COL)
- net COL9: now also MX_Num_*1.1 (COL), MX_Num_.1.1 (COL), MX_Num_/1.1 (COL), MX_Num_10.1 (COL), MX_Num_2.1 (COL), MX_Num_3.1 (COL), MX_Num_5.1 (COL), MX_Num_6.1 (COL), MX_Num_8.1 (COL), MX_Num_9.1 (COL)
- net LEDGND: now also R19.2, R20.2, R24.2, R25.2, R26.2, R27.2, R42.2, R44.2, R45.2, R73.2, R74.2, R75.2, R76.2, R78.2, R79.2, R80.2, R82.2, R89.2, R90.2, R91.2, R92.2, R16.2, R18.2, R43.2
- net ROW0: now also D19.1 (K), D21.1 (K)
- net ROW1: now also D18.1 (K), D20.1 (K)
- net ROW2: now also D26.1 (K), D28.1 (K)
- net ROW3: now also D25.1 (K), D27.1 (K)
- net ROW4: now also D43.1 (K), D45.1 (K)
- net ROW5: now also D44.1 (K), D46.1 (K)
- net ROW6: now also D75.1 (K), D77.1 (K)
- net ROW7: now also D76.1 (K), D78.1 (K)
- net ROW8: now also D80.1 (K), D82.1 (K), D85.1 (K), D92.1 (K), D94.1 (K); no longer D86.1 (K)
- net ROW9: now also D81.1 (K), D84.1 (K), D86.1 (K), D91.1 (K), D93.1 (K); no longer D85.1 (K)
- net at MX_Num_0_2U1.2 (ROW): now also D91.2 (A), MX_Num_11.2 (ROW)
- net at MX_Num_0_2U1.4 (LEDGND): now also MX_Num_11.4 (LEDGND), R89.1
- net at MX_LWIN7U1.2 (ROW): now also D84.2 (A), MX_LWIN1.2 (ROW)
- net at MX_LWIN7U1.3 (LED): now also MX_LWIN1.3 (LED)
- net at MX_LWIN7U1.4 (LEDGND): now also MX_LWIN1.4 (LEDGND), R82.1
- net at R42.1: now also MX_Num_4.4 (LEDGND)
- net at R45.1: now also MX_Num_+1.4 (LEDGND), MX_Num_+_2U1.4 (LEDGND)
- net at R26.1: now also MX_Num_3.4 (LEDGND)
- net at D19.2 (A): now also MX_Num_/1.2 (ROW)
- net at R78.1: now also MX_RALT1.4 (LEDGND), MX_RALT7U1.4 (LEDGND)
- net at MX_Num_L1.2 (ROW): now also D18.2 (A)
- net NLOCK_LEDGND: now reaches MX_Num_L1.4 (LEDGND)
- net NLOCK_LEDGND: now also R93.1
- net at D27.2 (A): now also MX_Num_3.2 (ROW)
- net at MX_Num_*1.2 (ROW): now also D20.2 (A)
- net at MX_Num_*1.4 (LEDGND): now also R19.1
- net at D28.2 (A): now also MX_Num_-2.2 (ROW)
- net at MX_Num_Enter_2U1.2 (ROW): now also D78.2 (A)
- net at MX_Num_Enter_2U1.4 (LEDGND): now also R76.1
- net at R80.1: now also MX_RWIN1.4 (LEDGND), MX_RWIN7U1.4 (LEDGND)
- net at D21.2 (A): now also MX_Num_-1.2 (ROW)
- net at R91.1: now also MX_Num_.1.4 (LEDGND)
- net at D75.2 (A): now also MX_Num_7.2 (ROW)
- net at MX_LCTRL7U1.2 (ROW): now also D83.2 (A), MX_LCTRL1.2 (ROW)
- net at MX_LCTRL7U1.4 (LEDGND): now also MX_LCTRL1.4 (LEDGND), R81.1
- net at MX_RWIN7U1.2 (ROW): now also D82.2 (A), MX_RWIN1.2 (ROW)
- net at D81.2 (A): now also MX_RFn1.2 (ROW)
- net at MX_Num_-1.4 (LEDGND): now also R20.1
- net at MX_Num_.1.2 (ROW): now also D93.2 (A)
- net at R44.1: now also MX_Num_6.4 (LEDGND)
- net at MX_Num_+1.2 (ROW): now also D46.2 (A), MX_Num_+_2U1.2 (ROW)
- net at MX_RFn1.4 (LEDGND): now also R79.1
- net at MX_Num_5.2 (ROW): now also D44.2 (A)
- net at MX_Num_5.4 (LEDGND): now also R43.1
- net at D80.2 (A): now also MX_RALT1.2 (ROW), MX_RALT7U1.2 (ROW)
- net at MX_Num_Macro2.2 (ROW): now also D94.2 (A), MX_Num_Macro1.2 (ROW)
- net at MX_Num_Macro2.4 (LEDGND): now also MX_Num_Macro1.4 (LEDGND), R92.1
- net at D87.2 (A), MX_RCTRL1.2 (ROW): now also MX_RCTRL7U1.2 (ROW)
- net at MX_Num_10.2 (ROW): now also D92.2 (A)
- net at MX_Num_10.4 (LEDGND): now also R90.1
- net at D45.2 (A): now also MX_Num_6.2 (ROW)
- net at R25.1: now also MX_Num_2.4 (LEDGND)
- net at D26.2 (A): now also MX_Num_2.2 (ROW)
- net at MX_Num_4.2 (ROW): now also D43.2 (A)
- net at D77.2 (A): now also MX_Num_9.2 (ROW)
- net at R75.1: now also MX_Num_9.4 (LEDGND)
- net at MX_Num_1.2 (ROW): now also D25.2 (A)
- net at MX_Num_1.4 (LEDGND): now also R24.1
- net at MX_Num_/1.4 (LEDGND): now also R18.1
- net at MX_Num_8.2 (ROW): now also D76.2 (A)
- net at MX_Num_8.4 (LEDGND): now also R74.1
- net at MX_RCTRL1.4 (LEDGND), R85.1: now also MX_RCTRL7U1.4 (LEDGND)
- net at D85.2 (A), MX_LALT1.2 (ROW): now also MX_LALT7U1.2 (ROW)
- net at MX_Num_7.4 (LEDGND): now also R73.1
- net at MX_LALT7U1.4 (LEDGND): now also MX_LALT1.4 (LEDGND), R83.1
- net at MX_Num_-2.4 (LEDGND): now also R27.1
- net SLOCK_IND renamed NLOCK_IND
- net SLOCK_LEDGND: no longer names the net of MX_HOME1.4 (LEDGND)
- net SLOCK_LEDGND: now also R16.1; no longer R93.1
Other:
- moved on the sheet: D80, MX_LALT7U1, MX_LCTRL7U1, MX_LWIN7U1, MX_Num_11, MX_Num_Macro2, MX_RALT1, MX_RALT7U1, MX_RCTRL7U1, MX_RWIN7U1, R78

Commit message: Updating pcb and schema
Schema: Fixed some of the schema issues in addition the matrix names require cleaning.
PCB: Switches has been aligned with the plate to make sure it have proper spacings.
Parts:
- MX_ENTR1: footprint MX_Alps_Hybrid:MX-2.5U-ReversedStabilizers -> MX_Alps_Hybrid:MX-2.25U-ReversedStabilizers
- MX_LWIN1: footprint MX_Alps_Hybrid:MX-1U -> MX_Alps_Hybrid:MX-1.25U
- MX_LWIN7U1, MX_RWIN7U1: footprint MX_Alps_Hybrid:MX-1.5U -> MX_Alps_Hybrid:MX-1U
Changed lines of the file:
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@@
       (effects (font (size 0.508 0.508)))
     )
-    (property "Footprint" "MX_Alps_Hybrid:MX-1.5U" (id 2) (at 77.089 176.403 0)
+    (property "Footprint" "MX_Alps_Hybrid:MX-1U" (id 2) (at 77.089 176.403 0)
       (effects (font (size 1.524 1.524)) hide)
     )
@@
       (effects (font (size 0.508 0.508)))
     )
-    (property "Footprint" "MX_Alps_Hybrid:MX-1.5U" (id 2) (at 253.365 176.911 0)
+    (property "Footprint" "MX_Alps_Hybrid:MX-1U" (id 2) (at 253.365 176.911 0)
       (effects (font (size 1.524 1.524)) hide)
     )
@@
       (effects (font (size 0.508 0.508)))
     )
-    (property "Footprint" "MX_Alps_Hybrid:MX-2.5U-ReversedStabilizers" (id 2) (at 268.097 106.299 0)
+    (property "Footprint" "MX_Alps_Hybrid:MX-2.25U-ReversedStabilizers" (id 2) (at 268.097 106.299 0)
       (effects (font (size 1.524 1.524)) hide)
     )
@@
       (effects (font (size 0.508 0.508)))
     )
-    (property "Footprint" "MX_Alps_Hybrid:MX-1U" (id 2) (at 77.089 150.749 0)
+    (property "Footprint" "MX_Alps_Hybrid:MX-1.25U" (id 2) (at 77.089 150.749 0)
       (effects (font (size 1.524 1.524)) hide)
     )

Commit message: Updating PCB
Added first row diodes and resistors to the pcb.
Note: there might be some clean up if there is no good tracing for diodes.
Parts:
- MX_LALT1, MX_LCTRL1, MX_LWIN1, MX_RALT1, MX_RCTRL1, MX_RFn1, MX_RWIN1: value MX-1.5U -> MX-1.25U
- MX_SP6.25U1: value MX-10U -> MX-6.25U
Changed lines of the file:
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@@
       (effects (font (size 1.524 1.524)))
     )
-    (property "Value" "MX-1.5U" (id 1) (at 256.8448 145.542 0)
+    (property "Value" "MX-1.25U" (id 1) (at 256.8448 145.542 0)
       (effects (font (size 0.508 0.508)))
     )
@@
       (effects (font (size 1.524 1.524)))
     )
-    (property "Value" "MX-1.5U" (id 1) (at 286.0548 146.304 0)
+    (property "Value" "MX-1.25U" (id 1) (at 286.0548 146.304 0)
       (effects (font (size 0.508 0.508)))
     )
@@
       (effects (font (size 1.524 1.524)))
     )
-    (property "Value" "MX-1.5U" (id 1) (at 271.3228 145.796 0)
+    (property "Value" "MX-1.25U" (id 1) (at 271.3228 145.796 0)
       (effects (font (size 0.508 0.508)))
     )
@@
       (effects (font (size 1.524 1.524)))
     )
-    (property "Value" "MX-1.5U" (id 1) (at 241.6048 145.288 0)
+    (property "Value" "MX-1.25U" (id 1) (at 241.6048 145.288 0)
       (effects (font (size 0.508 0.508)))
     )
@@
       (effects (font (size 1.524 1.524)))
     )
-    (property "Value" "MX-1.5U" (id 1) (at 95.0468 146.304 0)
+    (property "Value" "MX-1.25U" (id 1) (at 95.0468 146.304 0)
       (effects (font (size 0.508 0.508)))
     )
@@
       (effects (font (size 1.524 1.524)))
     )
-    (property "Value" "MX-10U" (id 1) (at 186.9948 147.574 0)
+    (property "Value" "MX-6.25U" (id 1) (at 186.9948 147.574 0)
       (effects (font (size 0.508 0.508)))
     )
@@
       (effects (font (size 1.524 1.524)))
     )
-    (property "Value" "MX-1.5U" (id 1) (at 110.7948 146.304 0)
+    (property "Value" "MX-1.25U" (id 1) (at 110.7948 146.304 0)
       (effects (font (size 0.508 0.508)))
     )
@@
       (effects (font (size 1.524 1.524)))
     )
-    (property "Value" "MX-1.5U" (id 1) (at 81.5848 146.304 0)
+    (property "Value" "MX-1.25U" (id 1) (at 81.5848 146.304 0)
       (effects (font (size 0.508 0.508)))
     )
