File: QMK 100 FRL/qfrl100.kicad_pcb (KiCad board)
At the start: 2 copper layers, 319 parts, among them J1 SM04B-SRSS-TB, J2 AVR-ISP-6, Q1 DSS60601MZ4-13, SW1 SW_PUSH, SW2 SW_SPDT, SW3 SW_SPDT, U1 ATmega32U4-MU, Y1 16MHz

Commit message: Updating pcb and schema
Schema: Fixed some of the schema issues in addition the matrix names require cleaning.
PCB: Switches has been aligned with the plate to make sure it have proper spacings.
Parts:
- C1, C2, C3, C4, C5, C6, C7, D1, D10, D11, D12, D13, D14, D15, D16, D17, D18, D19, D2, D20, D21, D22, D23, D24, D25, D26, D27, D28, D29, D3, D30, D31, D32, D33, D34, D35, D36, D37, D38, D39, D4, D40, D41, D42, D43, D44, D45, D46, D47, D48, D49, D5, D50, D51, D52, D53, D54, D55, D56, D57, D58, D59, D6, D60, D61, D62, D63, D64, D65, D66, D67, D68, D69, D7, D70, D71, D72, D73, D74, D75, D76, D77, D78, D79, D8, D80, D81, D82, D83, D84, D85, D86, D87, D88, D89, D9, D90, D91, D92, D93, D94, J1, J2, Q1, R1, R10, R11, R12, R13, R14, R15, R16, R17, R18, R19, R2, R20, R21, R22, R23, R24, R25, R26, R27, R28, R29, R3, R30, R31, R32, R33, R34, R35, R36, R37, R38, R39, R4, R40, R41, R42, R43, R44, R45, R46, R47, R48, R49, R5, R50, R51, R52, R53, R54, R55, R56, R57, R58, R59, R6, R60, R61, R62, R63, R64, R65, R66, R67, R68, R69, R7, R70, R71, R72, R73, R74, R75, R76, R77, R78, R79, R8, R80, R81, R82, R83, R84, R85, R86, R87, R88, R89, R9, R90, R91, R92, R93, R94, RC1, RC2, RC3, RC4, RC5, SW1, SW2, SW3, U1, Y1: moved to B.Cu
- MX_ENTR1: footprint MX_Alps_Hybrid:MX-2.5U-ReversedStabilizers -> MX_Alps_Hybrid:MX-2.25U-ReversedStabilizers
- MX_LWIN1: footprint MX_Alps_Hybrid:MX-1U -> MX_Alps_Hybrid:MX-1.25U
- MX_LWIN7U1, MX_RWIN7U1: footprint MX_Alps_Hybrid:MX-1.5U -> MX_Alps_Hybrid:MX-1U
- moved MX_LWIN1 812.1 mm to (108.6, 166.1)
- moved MX_5 801.1 mm to (177.6, 89.9)
- moved MX_4 800.0 mm to (158.6, 89.9)
- moved MX_A1 783.9 mm to (115.7, 128.0)
- moved MX_W1 752.5 mm to (130.0, 108.9)
- moved MX_1 740.6 mm to (101.4, 89.9)
- moved MX_LSHIFT2 733.9 mm to (94.3, 147.0)
- moved MX_X1 733.6 mm to (144.3, 147.0)
- moved MX_T1 732.0 mm to (187.2, 108.9)
- moved MX_K1 731.6 mm to (249.1, 128.0)
- moved MX_ESC1 706.8 mm to (82.4, 89.9)
- moved MX_M1 700.7 mm to (239.6, 147.0)
- moved MX_LSHIFT3 698.7 mm to (106.2, 147.0)
- moved MX_2 698.5 mm to (120.5, 89.9)
- moved MX_L1 692.4 mm to (268.1, 128.0)
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
Commit message: Updating PCB
Added first row diodes and resistors to the pcb.
Note: there might be some clean up if there is no good tracing for diodes.
Parts:
- MX_LALT1, MX_LCTRL1, MX_LWIN1, MX_RALT1, MX_RCTRL1, MX_RFn1, MX_RWIN1: value MX-1.5U -> MX-1.25U
- MX_SP6.25U1: value MX-10U -> MX-6.25U
- moved R20 305.3 mm to (484.2, 96.1), turned to -90 degrees
- moved R2 275.8 mm to (108.0, 96.1), turned to -90 degrees
- moved R18 269.6 mm to (446.9, 96.0), turned to -90 degrees
- moved D19 262.7 mm to (446.1, 89.6), turned to 90 degrees
- moved D2 261.3 mm to (109.5, 89.7), turned to 90 degrees
- moved R4 258.4 mm to (146.1, 96.1), turned to -90 degrees
- moved D20 255.5 mm to (465.1, 89.7), turned to 90 degrees
- moved R17 248.2 mm to (398.5, 96.0), turned to 90 degrees
- moved D21 238.7 mm to (484.2, 90.5), turned to 90 degrees
- moved D17 235.0 mm to (400.1, 89.6), turned to 90 degrees
- moved R6 224.5 mm to (184.2, 96.0), turned to -90 degrees
- moved D4 223.5 mm to (147.6, 89.7), turned to 90 degrees
- moved D1 221.1 mm to (90.5, 89.8), turned to 90 degrees
- moved R1 220.6 mm to (88.9, 96.0), turned to -90 degrees
- moved R19 215.4 mm to (465.1, 96.0), turned to -90 degrees
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
Commit message: Updating pcb
PCB diodes and resistor has been positioned near switch.

Next will be mcu and its components then tracing.
Parts:
- moved R28 305.2 mm to (93.7, 115.1), turned to 90 degrees
- moved D61 286.2 mm to (77.0, 146.8), turned to 90 degrees
- moved R27 278.4 mm to (479.4, 115.1), turned to -90 degrees
- moved R82 262.7 mm to (118.3, 172.3), turned to -90 degrees
- moved D27 262.6 mm to (465.1, 108.7), turned to 90 degrees
- moved D30 258.9 mm to (119.1, 108.7), turned to 90 degrees
- moved D83 253.0 mm to (95.2, 165.9), turned to 90 degrees
- moved R75 249.8 mm to (465.9, 153.2), turned to -90 degrees
- moved R83 244.9 mm to (142.1, 172.2), turned to -90 degrees
- moved D92 244.9 mm to (462.0, 165.9), turned to 90 degrees
- moved R24 242.2 mm to (441.3, 115.1), turned to -90 degrees
- moved D31 242.1 mm to (138.1, 108.7), turned to 90 degrees
- moved D29 238.1 mm to (95.2, 108.7), turned to 90 degrees
- moved D45 236.3 mm to (465.1, 127.7), turned to 90 degrees
- moved R48 236.1 mm to (160.3, 134.1), turned to -90 degrees
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
Commit message: Pcb update
Repositioned the remain components for the first design.
Parts:
- moved J1 86.2 mm to (365.9, 96.6), turned to 0 degrees
- moved J2 69.2 mm to (410.7, 128.6)
- moved C3 64.5 mm to (375.4, 127.8)
- moved RC3 62.7 mm to (375.4, 124.6)
- moved RC2 62.3 mm to (397.7, 134.1)
- moved RC1 59.4 mm to (379.4, 133.3)
- moved SW1 58.7 mm to (386.6, 129.4)
- moved Y1 56.8 mm to (375.9, 138.2)
- moved RC4 55.7 mm to (378.6, 124.6)
- moved Q1 52.7 mm to (397.7, 129.3)
- moved C1 52.0 mm to (376.2, 142.9)
- moved RC5 50.3 mm to (363.5, 137.3)
- moved C6 47.5 mm to (366.7, 150.8)
- moved C5 42.7 mm to (366.7, 147.6)
- moved C2 42.0 mm to (373.1, 142.9)
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